Commit message: 更改T265的碰撞体积，更改后T265可以正常工作，不再报找不到T265.stl的错误

File: legged_perceptive_description/urdf/sensor_t265.xacro (robot description, xacro)
@@ -38,5 +38,5 @@
                 <origin xyz="0 0 0" rpy="0 0 0"/>
                 <geometry>
-                    <mesh filename="package://realsense2_description/meshes/t265.stl"/>
+                    <box size="0.01 0.01 0.01"/>
                 </geometry>
             </collision>
