Commit message: 在mid360中增加Gazebo插件，在gazabo中模拟雷达数据

File: legged_perceptive_description/urdf/mid360.xacro (robot description, xacro)
@@ -2,5 +2,5 @@
 <robot xmlns:xacro="http://ros.org/wiki/xacro">
     <xacro:macro name="mid360"
-                 params="name parent *origin">
+                 params="name parent *origin ros_topic">
         <link name="${name}">
             <inertial>
@@ -61,8 +61,52 @@
             <child link="${name}"/>
         </joint>
+        <xacro:macro name="Livox_Mid_gazebo_sensor" params="name:=livox_laser">
         <gazebo reference="${name}">
-            <self_collide>1</self_collide>
-            <material>Gazebo/Blue</material>
-        </gazebo>
+        <sensor type="ray" name="laser_livox">
+            <pose>0 0 0.0 0 0 0</pose>
+            <visualize>true</visualize>
+            <always_on>True</always_on>
+            <update_rate>10</update_rate>
+            <!-- This ray plgin is only for visualization. -->
+            <plugin name="gazebo_ros_laser_controller" filename="liblivox_laser_simulation.so">
+                <ray>
+                <scan>
+                    <horizontal>
+                        <samples>100</samples>
+                        <resolution>1</resolution>
+                        <min_angle>-3.1415926535897931</min_angle>
+                <max_angle>3.1415926535897931</max_angle>
+                    </horizontal>
+                    <vertical>
+                        <samples>50</samples>
+                        <resolution>1</resolution>
+                        <min_angle>-0.122</min_angle>
+                <max_angle>0.908</max_angle>
+                    </vertical>
+                </scan>
+                <range>
+                    <min>0.1</min>
+                    <max>5</max>
+                    <resolution>1</resolution>
+                </range>
+                <noise>
+                    <type>gaussian</type>
+                    <mean>0.0</mean>
+                    <stddev>0.0</stddev>
+                </noise>
+                </ray>
+            <visualize>False</visualize>
+                <samples>20000</samples>
+                <downsample>1</downsample>
+                <csv_file_name>mid360.csv</csv_file_name>
+            <publish_pointcloud_type>2</publish_pointcloud_type>
+                <ros_topic>${ros_topic}</ros_topic>
+            <!-- <ros_topic>/livox/lidar</ros_topic>    -->
+            <frameName>base</frameName>
+            </plugin>
+        </sensor>
+    </gazebo>
+  </xacro:macro>
+    <xacro:Livox_Mid_gazebo_sensor name="${name}"/>
     </xacro:macro>
 </robot>

Commit message: 为Mid360增加Gazebo模型，并根据Mid360的实际范围对仿真角度进行更新

File: legged_perceptive_description/urdf/mid360.xacro (robot description, xacro)
@@ -3,4 +3,5 @@
     <xacro:macro name="mid360"
                  params="name parent *origin ros_topic frame">
+        <xacro:property name="M_PI" value="3.1415926535897931"/>
         <link name="${name}">
             <inertial>
@@ -13,9 +14,8 @@
             </inertial>
             <visual>
-                <origin rpy="0 0 0" xyz="0 0 -0.0076"/>
+                <origin rpy="${M_PI/2} 0 ${M_PI}" xyz="0 0 -0.0076"/>
                 <geometry>
-                    <sphere radius="0.022"/>
+                    <mesh filename="package://livox_laser_simulation/meshes/mid360.stl" scale="0.001 0.001 0.001"/>
                 </geometry>
-                <color rgba="0.0 0.0 0.5 0.5"/>
             </visual>
             <collision>
@@ -81,6 +81,6 @@
                         <samples>50</samples>
                         <resolution>1</resolution>
-                        <min_angle>-3.1415926535897931</min_angle>
-                <max_angle>3.1415926535897931</max_angle>
+                        <min_angle>-0.515</min_angle>
+                <max_angle>0.515</max_angle>
                     </vertical>
                 </scan>
@@ -97,4 +97,5 @@
                 </ray>
             <visualize>False</visualize>
+<!--            <visualize>True</visualize>-->
                 <samples>20000</samples>
                 <downsample>1</downsample>

Commit message: 更新Mid360到身体下，并取消Mid360碰撞模型（碰撞模型会让雷达存在很大的盲区，实机测试可以像宇树一样让支撑框架旋转起来消除盲区）

File: legged_perceptive_description/urdf/mid360.xacro (robot description, xacro)
@@ -19,40 +19,40 @@
                 </geometry>
             </visual>
-            <collision>
-                <origin xyz="0 0 0.027" rpy="0 0 0"/>
-                <geometry>
-                    <box size="0.003 0.067 0.0165"/>
-                </geometry>
-            </collision>
-            <collision>
-                <origin xyz="0 0.041 0.007" rpy="-1.04 0 0"/>
-                <geometry>
-                    <box size="0.003 0.055 0.024"/>
-                </geometry>
-            </collision>
-            <collision>
-                <origin xyz="0 -0.041 0.007" rpy="1.04 0 0"/>
-                <geometry>
-                    <box size="0.003 0.055 0.024"/>
-                </geometry>
-            </collision>
-            <collision>
-                <origin xyz="0 0 0.027" rpy="0 0 0"/>
-                <geometry>
-                    <box size="0.067 0.003 0.0165"/>
-                </geometry>
-            </collision>
-            <collision>
-                <origin xyz="0.041 0 0.007" rpy="0 1.04 0"/>
-                <geometry>
-                    <box size="0.055 0.003 0.024"/>
-                </geometry>
-            </collision>
-            <collision>
-                <origin xyz="-0.041 0 0.007" rpy="0 -1.04 0"/>
-                <geometry>
-                    <box size="0.055 0.003 0.024"/>
-                </geometry>
-            </collision>
+<!--            <collision>-->
+<!--                <origin xyz="0 0 0.027" rpy="0 0 0"/>-->
+<!--                <geometry>-->
+<!--                    <box size="0.003 0.067 0.0165"/>-->
+<!--                </geometry>-->
+<!--            </collision>-->
+<!--            <collision>-->
+<!--                <origin xyz="0 0.041 0.007" rpy="-1.04 0 0"/>-->
+<!--                <geometry>-->
+<!--                    <box size="0.003 0.055 0.024"/>-->
+<!--                </geometry>-->
+<!--            </collision>-->
+<!--            <collision>-->
+<!--                <origin xyz="0 -0.041 0.007" rpy="1.04 0 0"/>-->
+<!--                <geometry>-->
+<!--                    <box size="0.003 0.055 0.024"/>-->
+<!--                </geometry>-->
+<!--            </collision>-->
+<!--            <collision>-->
+<!--                <origin xyz="0 0 0.027" rpy="0 0 0"/>-->
+<!--                <geometry>-->
+<!--                    <box size="0.067 0.003 0.0165"/>-->
+<!--                </geometry>-->
+<!--            </collision>-->
+<!--            <collision>-->
+<!--                <origin xyz="0.041 0 0.007" rpy="0 1.04 0"/>-->
+<!--                <geometry>-->
+<!--                    <box size="0.055 0.003 0.024"/>-->
+<!--                </geometry>-->
+<!--            </collision>-->
+<!--            <collision>-->
+<!--                <origin xyz="-0.041 0 0.007" rpy="0 -1.04 0"/>-->
+<!--                <geometry>-->
+<!--                    <box size="0.055 0.003 0.024"/>-->
+<!--                </geometry>-->
+<!--            </collision>-->
         </link>
         <joint name="${name}_fixed" type="fixed">
@@ -70,4 +70,5 @@
             <!-- This ray plgin is only for visualization. -->
             <plugin name="gazebo_ros_laser_controller" filename="liblivox_laser_simulation.so">
+<!--            <plugin name='gazebo_ros_laser_controller' filename='libgazebo_ros_gpu_block_laser.so'>-->
                 <ray>
                 <scan>

File: legged_perceptive_description/urdf/robot.xacro (robot description, xacro)
@@ -6,15 +6,38 @@
     <xacro:include filename="$(find legged_perceptive_description)/urdf/sensor_t265.xacro"/>
     <xacro:include filename="$(find legged_perceptive_description)/urdf/mid360.xacro"/>
-        <xacro:sensor_d435 name="front_camera" topics_ns="front_camera" parent="base">
-            <origin xyz="0.36 -0.0 0.01" rpy="3.141 0.38 0"/>
-        </xacro:sensor_d435>
+    <xacro:sensor_d435 name="front_camera" topics_ns="front_camera" parent="base">
+<!--        <origin xyz="0.36 -0.0 0.01" rpy="3.141 0.38 0"/>-->
+        <origin xyz="0.30 -0.0 0.00" rpy="3.141 0.38 0"/>
+    </xacro:sensor_d435>
+    <xacro:sensor_d435 name="back_camera" topics_ns="back_camera" parent="base">
+        <origin xyz="-0.25 0.0 0.0" rpy="0 0.38 3.14"/>
+    </xacro:sensor_d435>
     <xacro:sensor_t265 name="tracking_camera" topics_ns="tracking_camera" parent="base">
         <origin xyz="0.16 0 0.085" rpy="0 -1.04 0"/>
     </xacro:sensor_t265>
     <xacro:mid360 name="livox_right" parent="base" ros_topic="/livox/lidar_192_168_8_101" frame="livox_right">
-        <origin xyz="0.365 -0.068 -0.030" rpy="0 0 0"/>
+<!--        up-->
+<!--        <origin xyz="0.335 -0.075 0.06" rpy="0.5 0.80 0"/>-->
+<!--        down-->
+<!--        <origin xyz="0.335 -0.068 -0.05" rpy="0 2.5 -0.5"/>-->
+<!--        middle-->
+<!--        <origin xyz="0.385 0 0.06" rpy="0 -2.3 0"/>&ndash;&gt;-->
+<!--        base-->
+        <origin xyz="0.12 0 -0.09" rpy="0 3.1415 0"/>
     </xacro:mid360>
-    <xacro:mid360 name="livox_left" parent="base" ros_topic="/livox/lidar_192_168_8_102" frame="livox_left">
-        <origin xyz="0.365 0.068 -0.030" rpy="0 0 0"/>
-    </xacro:mid360>
+<!--    <xacro:mid360 name="livox_left" parent="base" ros_topic="/livox/lidar_192_168_8_102" frame="livox_left">-->
+<!--&lt;!&ndash;        up&ndash;&gt;-->
+<!--        <origin xyz="0.335 0.075 0.06" rpy="-0.5 0.80 0"/>-->
+<!--&lt;!&ndash;        down&ndash;&gt;-->
+<!--&lt;!&ndash;        <origin xyz="0.335 0.068 -0.05" rpy="0 2.5 0.5"/>&ndash;&gt;-->
+<!--    </xacro:mid360>-->
+<!--    <xacro:mid360 name="livox_back" parent="base" ros_topic="/livox/lidar_192_168_8_103" frame="livox_back">-->
+<!--&lt;!&ndash;        up&ndash;&gt;-->
+<!--&lt;!&ndash;        <origin xyz="-0.243 0 0.1" rpy="0 -0.80 0"/>&ndash;&gt;-->
+<!--&lt;!&ndash;        down&ndash;&gt;-->
+<!--        <origin xyz="-0.283 0 -0.03" rpy="0 -3.14 0"/>-->
+<!--    </xacro:mid360>-->
+<!--    <xacro:mid360 name="livox_frontdown" parent="base" ros_topic="/livox/lidar_192_168_8_104" frame="livox_frontdown">-->
+<!--        <origin xyz="0.295 0 -0.05" rpy="0 2.5 0"/>-->
+<!--    </xacro:mid360>-->
 </robot>
